File: Rotary Switch Board.kicad_pcb (KiCad board)
At the start: 2 copper layers, 35.5 x 35.5 mm, 12 parts, among them J6 D2, SW1 1P8T_ROTARY_SWITCH

Commit message: added Silkscreen decorations
Other:
- board text added: "By NibbledPots"
- board text added: "Rotary Switch Board"
- board text added: "Single Output"
- board text added: "on Github"
Changed lines of the file:
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@@
       (outputformat 1)
       (mirror false)
-      (drillshape 1)
+      (drillshape 0)
       (scaleselection 1)
-      (outputdirectory "")
+      (outputdirectory "Gerbers/")
     )
   )
@@
   )
   (gr_circle (center 139.49 110.48) (end 146.32 94.07) (layer "Edge.Cuts") (width 0.1) (fill none))
+  (gr_text "on Github" (at 139.573 94.361) (layer "B.SilkS")
+    (effects (font (size 1 1) (thickness 0.15)) (justify mirror))
+  )
+  (gr_text "Single Output" (at 148.971 122.555 225) (layer "B.SilkS")
+    (effects (font (size 1 1) (thickness 0.15)) (justify mirror))
+  )
+  (gr_text "By NibbledPots" (at 148.717 98.171 315) (layer "B.SilkS")
+    (effects (font (size 1 1) (thickness 0.15)) (justify mirror))
+  )
+  (gr_text "Rotary Switch Board" (at 153.035 110.363 270) (layer "B.SilkS")
+    (effects (font (size 1 1) (thickness 0.15)) (justify mirror))
+  )
   (segment (start 126.915947 115.680775) (end 126.788947 115.680775) (width 0.254) (layer "F.Cu") (net 1))
   (segment (start 137.615114 108.599942) (end 137.615114 109.872734) (width 0.254) (layer "F.Cu") (net 1))

Commit message: Added GND planes
Routing:
- net GND: vias 0 -> 1
- added copper zone on B.Cu, net GND
- added copper zone on F.Cu, net GND
